File: Hackdeck/Hackdeck PCB/Bluprints.kicad_pcb (KiCad board)
At the start: 2 copper layers, 100 x 58 mm, 24 parts, among them J1 Conn_01x04, SW1 SW_Push, SW10 RotaryEncoder_Switch, SW2 SW_Push, SW3 SW_Push, SW4 SW_Push, SW5 SW_Push, SW6 SW_Push, SW7 SW_Push, SW8 SW_Push, U2 XIAO-RP2040-DIP

Commit message: Fix folders
Routing:
- net Col2: track 152.5 -> 155.0 mm
Changed lines of the file:
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@@
 	)
 	(segment
-		(start 139 69.399)
-		(end 138.411 69.399)
+		(start 143 83.69847)
+		(end 142.339 83.03747)
 		(width 0.2)
 		(layer "F.Cu")
@@
 	)
 	(segment
-		(start 130.54 97.92)
-		(end 140.601 87.859)
+		(start 139 69.399)
+		(end 138.411 69.399)
 		(width 0.2)
 		(layer "F.Cu")
@@
 	)
 	(segment
-		(start 140.601 87.859)
-		(end 140.601 69.751057)
+		(start 143 85.46)
+		(end 143 83.69847)
 		(width 0.2)
 		(layer "F.Cu")
@@
 	)
 	(segment
+		(start 143 72.150057)
+		(end 140.248943 69.399)
+		(width 0.2)
+		(layer "F.Cu")
+		(net 23)
+	)
+	(segment
 		(start 162.788892 60.199)
 		(end 139.801 60.199)
+		(width 0.2)
+		(layer "F.Cu")
+		(net 23)
+	)
+	(segment
+		(start 142.339 82.04253)
+		(end 143 81.38153)
 		(width 0.2)
 		(layer "F.Cu")
@@
 	)
 	(segment
+		(start 140.248943 69.399)
+		(end 139 69.399)
+		(width 0.2)
+		(layer "F.Cu")
+		(net 23)
+	)
+	(segment
 		(start 164.572892 61.983)
 		(end 162.788892 60.199)
@@
 	)
 	(segment
-		(start 140.601 69.751057)
-		(end 140.248943 69.399)
+		(start 130.54 97.92)
+		(end 143 85.46)
+		(width 0.2)
+		(layer "F.Cu")
+		(net 23)
+	)
+	(segment
+		(start 142.339 83.03747)
+		(end 142.339 82.04253)
 		(width 0.2)
 		(layer "F.Cu")
@@
 	)
 	(segment
-		(start 140.248943 69.399)
-		(end 139 69.399)
+		(start 143 81.38153)
+		(end 143 72.150057)
 		(width 0.2)
 		(layer "F.Cu")
